File: hardware/EAGLE/io.brd (EAGLE design)
At the start: 17.8 x 110.5 mm, 23 parts, among them J10 PJ301_THONKICONN6, J11 PJ301_THONKICONN6, J12 PJ301_THONKICONN6, J13 PJ301_THONKICONN6, J2 PJ301_THONKICONN6, J3 PJ301_THONKICONN6, J4 PJ301_THONKICONN6, J5 PJ301_THONKICONN6, J6 PJ301_THONKICONN6, J7 PJ301_THONKICONN6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

Commit message: up
Routing:
- net IO4A: track 12.5 -> 13.1 mm
Changed lines of the file:
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@@
 <layer number="17" name="Pads" color="2" fill="1" visible="yes" active="yes"/>
 <layer number="18" name="Vias" color="2" fill="1" visible="yes" active="yes"/>
-<layer number="19" name="Unrouted" color="6" fill="1" visible="yes" active="yes"/>
+<layer number="19" name="Unrouted" color="6" fill="1" visible="no" active="yes"/>
 <layer number="20" name="Dimension" color="24" fill="1" visible="yes" active="yes"/>
 <layer number="21" name="tPlace" color="7" fill="1" visible="yes" active="yes"/>
@@
 <layer number="38" name="bTest" color="7" fill="1" visible="no" active="yes"/>
 <layer number="39" name="tKeepout" color="4" fill="11" visible="yes" active="yes"/>
-<layer number="40" name="bKeepout" color="1" fill="11" visible="yes" active="yes"/>
-<layer number="41" name="tRestrict" color="4" fill="10" visible="yes" active="yes"/>
-<layer number="42" name="bRestrict" color="1" fill="10" visible="yes" active="yes"/>
+<layer number="40" name="bKeepout" color="1" fill="11" visible="no" active="yes"/>
+<layer number="41" name="tRestrict" color="4" fill="10" visible="no" active="yes"/>
+<layer number="42" name="bRestrict" color="1" fill="10" visible="no" active="yes"/>
 <layer number="43" name="vRestrict" color="2" fill="10" visible="no" active="yes"/>
 <layer number="44" name="Drills" color="7" fill="1" visible="no" active="yes"/>
@@
 </element>
 <element name="J2" library="og-pj301_variations" package="WQP_PJ_301M6" value="PJ301_THONKICONN6" x="15.24" y="113.3475" smashed="yes" rot="MR0">
-<attribute name="NAME" x="-54.03" y="232.8075" size="1.27" layer="26" rot="MR180"/>
+<attribute name="NAME" x="12.01" y="118.5075" size="1.27" layer="26" rot="MR180"/>
 </element>
 <element name="J3" library="og-pj301_variations" package="WQP_PJ_301M6" value="PJ301_THONKICONN6" x="5.08" y="113.3475" smashed="yes" rot="MR0">
@@
 <wire x1="14.0208" y1="80.772" x2="13.716" y2="81.0768" width="0.4064" layer="16"/>
 <wire x1="14.0208" y1="75.8952" x2="14.0208" y2="80.772" width="0.4064" layer="16"/>
-<wire x1="16.1544" y1="75.8952" x2="14.0208" y2="75.8952" width="0.4064" layer="1"/>
-<wire x1="16.4592" y1="75.5904" x2="16.1544" y2="75.8952" width="0.4064" layer="1"/>
-<wire x1="17.3736" y1="75.5904" x2="16.4592" y2="75.5904" width="0.4064" layer="1"/>
+<wire x1="17.3736" y1="75.5904" x2="14.3256" y2="75.5904" width="0.4064" layer="1"/>
+<wire x1="14.3256" y1="75.5904" x2="14.0208" y2="75.8952" width="0.4064" layer="1"/>
 <wire x1="18.5928" y1="76.8096" x2="17.3736" y2="75.5904" width="0.4064" layer="1"/>
 <wire x1="18.5928" y1="78.3336" x2="18.5928" y2="76.8096" width="0.4064" layer="1"/>
@@
 <contactref element="SV1" pad="5"/>
 <wire x1="15.24" y1="92.6592" x2="16.4592" y2="92.6592" width="0.4064" layer="1"/>
-<wire x1="13.1064" y1="90.5256" x2="15.24" y2="92.6592" width="0.4064" layer="1"/>
-<wire x1="11.2776" y1="90.5256" x2="13.1064" y2="90.5256" width="0.4064" layer="1"/>
-<wire x1="10.9728" y1="90.2208" x2="11.2776" y2="90.5256" width="0.4064" layer="1"/>
-<wire x1="10.3632" y1="90.2208" x2="10.9728" y2="90.2208" width="0.4064" layer="1"/>
+<wire x1="12.8016" y1="90.2208" x2="15.24" y2="92.6592" width="0.4064" layer="1"/>
+<wire x1="10.3632" y1="90.2208" x2="12.8016" y2="90.2208" width="0.4064" layer="1"/>
 <wire x1="16.4592" y1="92.6592" x2="16.51" y2="92.71" width="0.4064" layer="1"/>
 <wire x1="10.3632" y1="90.2208" x2="10.16" y2="90.17" width="0.4064" layer="1"/>
@@
 <wire x1="12.4968" y1="13.1064" x2="12.4968" y2="11.5824" width="0.4064" layer="1"/>
 <wire x1="11.8872" y1="13.716" x2="12.4968" y2="13.1064" width="0.4064" layer="1"/>
-<wire x1="11.8872" y1="17.3736" x2="11.8872" y2="13.716" width="0.4064" layer="1"/>
-<wire x1="15.24" y1="20.7264" x2="11.8872" y2="17.3736" width="0.4064" layer="1"/>
-<wire x1="15.24" y1="22.225" x2="15.24" y2="20.7264" width="0.4064" layer="1"/>
+<wire x1="11.8872" y1="19.9136" x2="11.8872" y2="13.716" width="0.4064" layer="1"/>
+<wire x1="15.24" y1="22.225" x2="14.1986" y2="22.225" width="0.4064" layer="1"/>
+<wire x1="14.1986" y1="22.225" x2="11.8872" y2="19.9136" width="0.4064" layer="1"/>
 <wire x1="12.4968" y1="11.5824" x2="12.7" y2="11.43" width="0.4064" layer="1"/>
 </signal>
@@
 <wire x1="7.62" y1="13.4112" x2="7.62" y2="11.43" width="0.4064" layer="1"/>
 <wire x1="7.0104" y1="14.0208" x2="7.62" y2="13.4112" width="0.4064" layer="1"/>
-<wire x1="7.0104" y1="18.8976" x2="7.0104" y2="14.0208" width="0.4064" layer="1"/>
-<wire x1="4.8768" y1="21.0312" x2="7.0104" y2="18.8976" width="0.4064" layer="1"/>
-<wire x1="5.1816" y1="21.336" x2="4.8768" y2="21.0312" width="0.4064" layer="1"/>
-<wire x1="5.1816" y1="21.9456" x2="5.1816" y2="21.336" width="0.4064" layer="1"/>
-<wire x1="5.1816" y1="21.9456" x2="5.08" y2="22.225" width="0.4064" layer="1"/>
+<wire x1="7.0104" y1="20.1676" x2="7.0104" y2="14.0208" width="0.4064" layer="1"/>
+<wire x1="5.152571875" y1="22.025428125" x2="7.0104" y2="20.1676" width="0.4064" layer="1"/>
+<wire x1="5.152571875" y1="22.025428125" x2="5.08" y2="22.225" width="0.4064" layer="1"/>
 </signal>
 <signal name="BUTTON">
