File: hardware/EAGLE/pcb.brd (EAGLE design)
At the start: 17.8 x 110.5 mm, 41 parts, among them IC1 4017N, IC2 DG412DJD, IC3 DG412DJD, Q1 MMBT3904, Q2 MMBT3904, Q3 MMBT3904, Q4 MMBT3904

Commit message: eagle
Parts:
- moved D2 0.64 mm to (3.81, 72.4)
- moved D1 0.63 mm to (16.5, 72.4)
Routing:
- net N$1: track 42.2 -> 8.62 mm, vias 7 -> 0
- net GND: track 238.4 -> 216.8 mm, vias 2 -> 5
- net N$5: track 94.6 -> 112.0 mm, vias 2 -> 6
- net +12V: track 156.9 -> 144.7 mm, vias 2 -> 8
- net N$7: track 70.9 -> 59.8 mm, vias 0 -> 4
- net N$3: track 82.1 -> 86.9 mm, vias 5 -> 8
- net N$10: track 67.8 -> 72.0 mm, vias 4 -> 0
- net N$9: track 75.2 -> 71.9 mm, vias 6 -> 4
- net N$19: track 10.1 -> 13.2 mm
- net N$11: track 71.0 -> 73.7 mm
- net NO: track 52.8 -> 54.0 mm, vias 1 -> 2
- net RES: track 77.8 -> 78.9 mm, vias 1 -> 6
- net STEP: track 4.03 -> 3.05 mm, vias 1 -> 0
- net N$6: track 62.4 -> 61.4 mm, vias 4 -> 6
- net N$2: track 10.2 -> 9.38 mm
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- added copper zone on layer 1, net GND
- added copper zone on layer 16, net GND

Commit message: FINALIZED PCBs
Parts:
- added C6: 100n, rcl:C0603
- added D7: 1N4148WT, diode:SOD523
- added R19: 10k, rcl:R0603
- moved C1 0.95 mm to (17.1, 58.7)
- moved D6 0.32 mm to (17.8, 51.1)
Connections:
- removed net N$33: SV2.6
- new net BUTTON: R19.1, SV2.6
- new net N$13: C6.1, D7.A, R19.2
- net +12V: now also SV2.9
- net CLK: now also D7.C
- net GND: now also C6.2; no longer SV2.9
Routing:
- net N$13: track 0.00 -> 56.7 mm, vias 0 -> 2
- net N$10: track 72.0 -> 104.3 mm, vias 0 -> 4
- net N$20: track 8.85 -> 35.4 mm
- net N$5: track 112.0 -> 93.9 mm, vias 6 -> 4
- net GND: track 216.8 -> 199.6 mm, vias 5 -> 7
- net Q1: track 83.9 -> 100.4 mm, vias 3 -> 6
- net Q0: track 84.5 -> 95.0 mm, vias 2 -> 4
- net +12V: track 144.7 -> 136.7 mm, vias 8 -> 7
- net N$6: track 61.4 -> 67.3 mm, vias 6 -> 4
- net N$12: track 11.8 -> 17.5 mm
- net BUTTON: track 0.00 -> 5.50 mm
- net NO: track 54.0 -> 59.0 mm, vias 2 -> 4
- net N$19: track 13.2 -> 8.58 mm, vias 0 -> 2
- net N$3: track 86.9 -> 82.9 mm, vias 8 -> 2
- net -12V: track 71.2 -> 67.4 mm, vias 4 -> 3
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- added copper zone on layer 1, net N$18
- added copper zone on layer 16, net N$22
- removed copper zone on layer 1, net GND
- removed copper zone on layer 16, net GND

Commit message: Submitted for Artist
and quick fixed layer errors
Routing:
- added copper zone on layer 1, net GND
- added copper zone on layer 16, net GND
- removed copper zone on layer 1, net N$18
- removed copper zone on layer 16, net N$22
Changed lines of the file:
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@@
 <via x="12.065" y="54.76875" extent="1-16" drill="0.3"/>
 <via x="13.6525" y="73.66" extent="1-16" drill="0.3"/>
+<polygon width="0.4064" layer="16">
+<vertex x="1.27" y="119.38"/>
+<vertex x="19.05" y="119.38"/>
+<vertex x="19.05" y="8.89"/>
+<vertex x="1.27" y="8.89"/>
+</polygon>
+<polygon width="0.4064" layer="1">
+<vertex x="1.27" y="119.38"/>
+<vertex x="19.05" y="119.38"/>
+<vertex x="19.05" y="8.89"/>
+<vertex x="1.27" y="8.89"/>
+</polygon>
 </signal>
 <signal name="BUTTON">
@@
 <via x="6.19125" y="94.45625" extent="1-16" drill="0.3"/>
 </signal>
-<signal name="N$18">
-<polygon width="0.4064" layer="1">
-<vertex x="1.27" y="119.38"/>
-<vertex x="19.05" y="119.38"/>
-<vertex x="19.05" y="8.89"/>
-<vertex x="1.27" y="8.89"/>
-</polygon>
-</signal>
-<signal name="N$22">
-<polygon width="0.4064" layer="16">
-<vertex x="1.27" y="119.38"/>
-<vertex x="19.05" y="119.38"/>
-<vertex x="19.05" y="8.89"/>
-<vertex x="1.27" y="8.89"/>
-</polygon>
-</signal>
 </signals>

Commit message: Added BOM
And buffer caps, and refined design
Parts:
- added C7, C8: 10u, rcl:153CLV-0605
- J1: value (none) -> 2x5 pin header
- SV1, SV2: value (none) -> 1x10 pin header
- SV3: value (none) -> 1x3 pin header
Connections:
- net +12V: now also C7.+
- net -12V: now also C8.-
- net GND: now also C7.-, C8.+
Routing:
- net N$10: track 104.3 -> 74.9 mm
- net N$20: track 35.4 -> 8.85 mm
- net +12V: track 136.7 -> 158.0 mm, vias 7 -> 4
- net N$5: track 93.9 -> 114.9 mm, vias 4 -> 6
- net Q3: track 106.2 -> 125.9 mm, vias 6 -> 4
- net GND: track 199.6 -> 214.6 mm, vias 7 -> 6
- net Q0: track 95.0 -> 84.0 mm
- net N$13: track 56.7 -> 49.7 mm, vias 2 -> 4
- net N$12: track 17.5 -> 11.8 mm
- net -12V: track 67.4 -> 72.7 mm
- net Q1: track 100.4 -> 95.5 mm, vias 6 -> 4
- net CLK: track 77.5 -> 82.2 mm, vias 2 -> 4
- net N$19: track 8.58 -> 13.2 mm, vias 2 -> 0
- net N$9: track 73.5 -> 77.6 mm, vias 2 -> 4
- net N$3: track 82.9 -> 86.8 mm, vias 2 -> 6
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