File: hardware/EAGLE/io.sch (EAGLE design)
At the start: 21 parts, among them J10 PJ301_THONKICONN6, J11 PJ301_THONKICONN6, J12 PJ301_THONKICONN6, J13 PJ301_THONKICONN6, J2 PJ301_THONKICONN6, J3 PJ301_THONKICONN6, J4 PJ301_THONKICONN6, J5 PJ301_THONKICONN6, J6 PJ301_THONKICONN6, J7 PJ301_THONKICONN6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

Commit message: FINALIZED PCBs
Parts:
- added SW1: (no value), SparkFun:TAC_SWITCHPTH
Connections:
- removed net N$33: SV2.6
- new net +12V: SV2.9, SW1.1, SW1.2
- new net BUTTON: SV2.6, SW1.3, SW1.4
- net GND: no longer SV2.9
Changed lines of the file:
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@@
 <?xml version="1.0" encoding="utf-8"?>
 <!DOCTYPE eagle SYSTEM "eagle.dtd">
-<eagle version="9.5.2">
+<eagle version="9.2.2">
 <drawing>
 <settings>
@@
 <classes>
 <class number="0" name="default" width="0.4064" drill="0">
-<clearance class="0" value="0.1016"/>
+<clearance class="0" value="0.2032"/>
 </class>
 </classes>
@@
 <part name="SV3" library="con-lstb" library_urn="urn:adsk.eagle:library:162" deviceset="MA03-1" device="" package3d_urn="urn:adsk.eagle:package:8339/1"/>
 <part name="GND2" library="supply1" library_urn="urn:adsk.eagle:library:371" deviceset="GND" device=""/>
+<part name="SW1" library="SparkFun" deviceset="TAC_SWITCH" device="PTH"/>
 </parts>
 <sheets>
@@
 <attribute name="VALUE" x="-160.02" y="-25.4" size="1.778" layer="96"/>
 </instance>
+<instance part="SW1" gate="S" x="-157.48" y="55.88" smashed="yes">
+<attribute name="NAME" x="-160.02" y="62.23" size="1.778" layer="95"/>
+<attribute name="VALUE" x="-160.02" y="49.53" size="1.778" layer="96"/>
+</instance>
 </instances>
 <busses>
@@
 <pinref part="SV1" gate="1" pin="9"/>
 <label x="-175.26" y="25.4" size="1.778" layer="95" rot="R180"/>
-</segment>
-<segment>
-<wire x1="-139.7" y1="25.4" x2="-142.24" y2="25.4" width="0.1524" layer="91"/>
-<pinref part="SV2" gate="1" pin="9"/>
-<label x="-139.7" y="25.4" size="1.778" layer="95"/>
 </segment>
 </net>
@@
 </segment>
 </net>
-<net name="N$33" class="0">
+<net name="BUTTON" class="0">
 <segment>
 <wire x1="-139.7" y1="17.78" x2="-142.24" y2="17.78" width="0.1524" layer="91"/>
@@
 <label x="-139.7" y="17.78" size="1.778" layer="95"/>
 </segment>
+<segment>
+<pinref part="SW1" gate="S" pin="4"/>
+<wire x1="-152.4" y1="53.34" x2="-149.86" y2="53.34" width="0.1524" layer="91"/>
+<wire x1="-149.86" y1="53.34" x2="-149.86" y2="55.88" width="0.1524" layer="91"/>
+<pinref part="SW1" gate="S" pin="3"/>
+<wire x1="-149.86" y1="55.88" x2="-152.4" y2="55.88" width="0.1524" layer="91"/>
+<wire x1="-149.86" y1="55.88" x2="-147.32" y2="55.88" width="0.1524" layer="91"/>
+<junction x="-149.86" y="55.88"/>
+<label x="-147.32" y="55.88" size="1.778" layer="95"/>
+</segment>
 </net>
 <net name="STEP" class="0">
@@
 </segment>
 </net>
+<net name="+12V" class="0">
+<segment>
+<wire x1="-139.7" y1="25.4" x2="-142.24" y2="25.4" width="0.1524" layer="91"/>
+<pinref part="SV2" gate="1" pin="9"/>
+<label x="-139.7" y="25.4" size="1.778" layer="95"/>
+</segment>
+<segment>
+<pinref part="SW1" gate="S" pin="1"/>
+<wire x1="-162.56" y1="55.88" x2="-165.1" y2="55.88" width="0.1524" layer="91"/>
+<pinref part="SW1" gate="S" pin="2"/>
+<wire x1="-165.1" y1="55.88" x2="-165.1" y2="53.34" width="0.1524" layer="91"/>
+<wire x1="-165.1" y1="53.34" x2="-162.56" y2="53.34" width="0.1524" layer="91"/>
+<wire x1="-165.1" y1="55.88" x2="-167.64" y2="55.88" width="0.1524" layer="91"/>
+<junction x="-165.1" y="55.88"/>
+<label x="-167.64" y="55.88" size="1.778" layer="95" rot="R180"/>
+</segment>
+</net>
 </nets>
 </sheet>
 </sheets>
+<errors>
+</errors>
 </schematic>
 </drawing>

Commit message: Added BOM
And buffer caps, and refined design
Parts:
- SV1, SV2: value (none) -> 1x10 pin header
- SV3: value (none) -> 1x3 pin header
- SW1: value (none) -> SPDT On-Off-On
Changed lines of the file:
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@@
 <part name="D3" library="SparkFun-LED" deviceset="LED" device="3MM"/>
 <part name="D4" library="SparkFun-LED" deviceset="LED" device="3MM"/>
-<part name="SV1" library="con-lstb" library_urn="urn:adsk.eagle:library:162" deviceset="MA10-1" device="" package3d_urn="urn:adsk.eagle:package:8346/1"/>
-<part name="SV2" library="con-lstb" library_urn="urn:adsk.eagle:library:162" deviceset="MA10-1" device="" package3d_urn="urn:adsk.eagle:package:8346/1"/>
+<part name="SV1" library="con-lstb" library_urn="urn:adsk.eagle:library:162" deviceset="MA10-1" device="" package3d_urn="urn:adsk.eagle:package:8346/1" value="1x10 pin header"/>
+<part name="SV2" library="con-lstb" library_urn="urn:adsk.eagle:library:162" deviceset="MA10-1" device="" package3d_urn="urn:adsk.eagle:package:8346/1" value="1x10 pin header"/>
 <part name="S1" library="SparkFun-Switches" deviceset="SWITCH-SPDT" device="-PTH-11.6X4.0MM-SHORT_LEADS"/>
 <part name="GND1" library="supply1" library_urn="urn:adsk.eagle:library:371" deviceset="GND" device=""/>
 <part name="R1" library="rcl" library_urn="urn:adsk.eagle:library:334" deviceset="R-US_" device="R0603" package3d_urn="urn:adsk.eagle:package:23555/3" value="1k"/>
-<part name="SV3" library="con-lstb" library_urn="urn:adsk.eagle:library:162" deviceset="MA03-1" device="" package3d_urn="urn:adsk.eagle:package:8339/1"/>
+<part name="SV3" library="con-lstb" library_urn="urn:adsk.eagle:library:162" deviceset="MA03-1" device="" package3d_urn="urn:adsk.eagle:package:8339/1" value="1x3 pin header"/>
 <part name="GND2" library="supply1" library_urn="urn:adsk.eagle:library:371" deviceset="GND" device=""/>
-<part name="SW1" library="SparkFun" deviceset="TAC_SWITCH" device="PTH"/>
+<part name="SW1" library="SparkFun" deviceset="TAC_SWITCH" device="PTH" value="SPDT On-Off-On"/>
 </parts>
 <sheets>
@@
 <instance part="SW1" gate="S" x="-157.48" y="55.88" smashed="yes">
 <attribute name="NAME" x="-160.02" y="62.23" size="1.778" layer="95"/>
-<attribute name="VALUE" x="-160.02" y="49.53" size="1.778" layer="96"/>
+<attribute name="VALUE" x="-162.56" y="49.53" size="1.778" layer="96"/>
 </instance>
 </instances>
