File: hardware/EAGLE/panel.brd (EAGLE design)
At the start: 20 x 128.5 mm, 1 part

Commit message: FINALIZED PCBs
Changed lines of the file:
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@@
 <?xml version="1.0" encoding="utf-8"?>
 <!DOCTYPE eagle SYSTEM "eagle.dtd">
-<eagle version="9.5.2">
+<eagle version="9.2.2">
 <drawing>
 <settings>
@@
 <layer number="43" name="vRestrict" color="2" fill="10" visible="no" active="yes"/>
 <layer number="44" name="Drills" color="7" fill="1" visible="no" active="yes"/>
-<layer number="45" name="Holes" color="7" fill="1" visible="no" active="yes"/>
+<layer number="45" name="Holes" color="7" fill="1" visible="yes" active="yes"/>
 <layer number="46" name="Milling" color="3" fill="1" visible="no" active="yes"/>
-<layer number="47" name="Measures" color="7" fill="1" visible="no" active="yes"/>
+<layer number="47" name="Measures" color="7" fill="1" visible="yes" active="yes"/>
 <layer number="48" name="Document" color="7" fill="1" visible="no" active="yes"/>
 <layer number="49" name="Reference" color="7" fill="1" visible="no" active="yes"/>
@@
 <hole x="12.3825" y="78.74" drill="3.0226"/>
 <hole x="16.8275" y="78.74" drill="3.0226"/>
+<hole x="10.16" y="102.87" drill="5.0038"/>
 </plain>
 <attributes>

Commit message: Added BOM
And buffer caps, and refined design
Routing:
- added copper zone on layer 16, net GND
Changed lines of the file:
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@@
 <board>
 <plain>
-<hole x="10.16" y="87.63" drill="6.985"/>
+<hole x="10.16" y="87.63" drill="5.0038"/>
 <hole x="5.08" y="55.88" drill="6.0198"/>
 <hole x="15.24" y="55.88" drill="6.0198"/>
@@
 <vertex x="0" y="128.27"/>
 <vertex x="20.32" y="128.27"/>
+<vertex x="20.32" y="0"/>
+<vertex x="0" y="0"/>
+</polygon>
+<polygon width="0.1524" layer="16">
+<vertex x="0" y="128.27"/>
+<vertex x="20.32" y="128.27"/>
