File: hardware/EAGLE/pcb.sch (EAGLE design)
At the start: 40 parts, among them IC1 4017N, IC2 DG412DJD, IC3 DG412DJD, Q1 MMBT3904, Q2 MMBT3904, Q3 MMBT3904, Q4 MMBT3904

Commit message: FINALIZED PCBs
Parts:
- added C6: 100n, rcl:C-USC0603
- added D7: 1N4148WT, diode:DIODE-SOD523
- added R19: 10k, rcl:R-US_R0603
Connections:
- removed net N$33: SV2.6
- new net BUTTON: R19.1, SV2.6
- new net N$13: C6.1, D7.A, R19.2
- net +12V: now also SV2.9
- net CLK: now also D7.C
- net GND: now also C6.2; no longer SV2.9
Other:
- moved on the sheet: SV1, SV2, SV3

Commit message: Added BOM
And buffer caps, and refined design
Parts:
- added C7, C8: 10u, rcl:CPOL-EU153CLV-0605
- J1: value (none) -> 2x5 pin header
- SV1, SV2: value (none) -> 1x10 pin header
- SV3: value (none) -> 1x3 pin header
Connections:
- net +12V: now also C7.+
- net -12V: now also C8.-
- net GND: now also C7.-, C8.+
